Commit message: update mm_moveit_config package(Dv-PC)

File: mm_description/urdf/mobile_manipulator.gazebo.xacro (robot description, xacro)
@@ -36,9 +36,9 @@
           <frameName>${name}_optical_frame</frameName>
           <pointCloudCutoff>0.5</pointCloudCutoff>
-          <distortionK1>0.00000001</distortionK1>
-          <distortionK2>0.00000001</distortionK2>
-          <distortionK3>0.00000001</distortionK3>
-          <distortionT1>0.00000001</distortionT1>
-          <distortionT2>0.00000001</distortionT2>
+          <distortionK1>0.0000000</distortionK1>
+          <distortionK2>0.0000000</distortionK2>
+          <distortionK3>0.0000000</distortionK3>
+          <distortionT1>0.0000000</distortionT1>
+          <distortionT2>0.0000000</distortionT2>
           <CxPrime>0</CxPrime>
           <Cx>0</Cx>
@@ -74,9 +74,9 @@
           <frameName>${name}_optical_frame</frameName>
           <pointCloudCutoff>0.5</pointCloudCutoff>
-          <distortionK1>0.00000001</distortionK1>
-          <distortionK2>0.00000001</distortionK2>
-          <distortionK3>0.00000001</distortionK3>
-          <distortionT1>0.00000001</distortionT1>
-          <distortionT2>0.00000001</distortionT2>
+          <distortionK1>0.0000000</distortionK1>
+          <distortionK2>0.0000000</distortionK2>
+          <distortionK3>0.0000000</distortionK3>
+          <distortionT1>0.0000000</distortionT1>
+          <distortionT2>0.0000000</distortionT2>
           <CxPrime>0</CxPrime>
           <Cx>0</Cx>

File: mm_description/urdf/mobile_manipulator.urdf (robot description, URDF)
Before this commit: robot mm, 17 links, 16 joints
Links:
- removed link xtion_link
- added link xtion1_frame, mass 1e-5
Joints:
- removed joint arm_base_link_2_xtion_link
- added joint arm_base_link_2_xtion1_frame: type fixed, parent arm_base_link, child xtion1_frame, origin xyz=-0.3541575 0.1507695 0.779517 rpy=-0.369 0.825 1.119

File: mm_description/urdf/mobile_manipulator.urdf.xacro (robot description, xacro)
@@ -27,5 +27,5 @@
         <inertia ixx="1e-6" ixy="0" ixz="0" iyy="1e-6" iyz="0" izz="1e-6" />
       </inertial>
-      <visual>
+      <!--visual>
         <origin xyz="0.02 -0.03 0" rpy="1.57 0 1.57" />
         <geometry>
@@ -38,5 +38,5 @@
            <mesh filename="package://mm_description/meshes/sensors/asus_xtion_pro_live_camera.dae" scale="0.001 0.001 0.001"/>
         </geometry>
-      </collision >
+      </collision -->
   </link>
   <joint name="${arm_prefix}base_link_2_xtion1_frame" type="fixed">

Commit message: add a xtion1_optical_frame link in xacro file of mobile manipulator, able to show point cloud of xtion on rviz.

File: mm_description/urdf/mobile_manipulator.gazebo.xacro (robot description, xacro)
@@ -35,4 +35,5 @@
           <pointCloudTopicName>${name}/depth/points</pointCloudTopicName>
           <frameName>${name}_optical_frame</frameName>
+          <!--frameName>${name}_frame</frameName-->
           <pointCloudCutoff>0.5</pointCloudCutoff>
           <distortionK1>0.0000000</distortionK1>
@@ -73,4 +74,5 @@
           <pointCloudTopicName>${name}/rgb/points</pointCloudTopicName>
           <frameName>${name}_optical_frame</frameName>
+          <!--frameName>${name}_frame</frameName-->
           <pointCloudCutoff>0.5</pointCloudCutoff>
           <distortionK1>0.0000000</distortionK1>

File: mm_description/urdf/mobile_manipulator.urdf.xacro (robot description, xacro)
@@ -38,5 +38,5 @@
            <mesh filename="package://mm_description/meshes/sensors/asus_xtion_pro_live_camera.dae" scale="0.001 0.001 0.001"/>
         </geometry>
-      </collision -->
+      </collision-->
   </link>
   <joint name="${arm_prefix}base_link_2_xtion1_frame" type="fixed">
@@ -45,4 +45,10 @@
 	<origin xyz="-0.3541575 0.1507695 0.779517" rpy="-0.369 0.825 1.119"/>
   </joint>
+  <joint name="xtion1_frame_2_xtion1_optical_frame" type="fixed">
+    <parent link="xtion1_frame" />
+    <child link="xtion1_optical_frame" />
+    <origin xyz="0 0 0" rpy="${-M_PI/2} 0 ${-M_PI/2}" />
+  </joint>
+  <link name="xtion1_optical_frame" />
   <xacro:kinect_camera_gazebo_v0 name="xtion1" />
 </robot>
