Commit message: change the folder structure of mm_description/urdf

File: mm_description/urdf/mobile_manipulator.urdf.xacro (robot description, xacro)
@@ -6,7 +6,7 @@
   <xacro:include filename="$(find mm_description)/urdf/common.gazebo" />
   <!-- ur5 -->
-  <xacro:include filename="$(find mm_description)/urdf/ur5.urdf.xacro" />
+  <xacro:include filename="$(find mm_description)/urdf/ur5/ur5.urdf.xacro" />
   <!-- mobile base -->
-  <xacro:include filename="$(find mm_description)/urdf/mobile_base.xacro" />
+  <xacro:include filename="$(find mm_description)/urdf/mobile_base/mobile_base.xacro" />
   <!-- arm -->
   <xacro:ur5_robot prefix="${arm_prefix}" joint_limited="true"/>
@@ -22,5 +22,5 @@
   <joint name="base_link_2_${arm_prefix}base_link" type="fixed">
     <parent link="base_link" />
-    <child link="arm_base_link" />
+    <child link="${arm_prefix}base_link" />
     <origin xyz="0.40 0 0.823" rpy="0 0 -1.5708" />
   </joint>
@@ -34,5 +34,5 @@
         <origin xyz="0.02 -0.03 0" rpy="1.57 0 1.57" />
         <geometry>
-          <mesh filename="package://mm_description/meshes/mobile_base/asus_xtion_pro_live_camera.dae" scale="0.001 0.001 0.001"/>
+          <mesh filename="package://mm_description/meshes/sensors/asus_xtion_pro_live_camera.dae" scale="0.001 0.001 0.001"/>
         </geometry>
       </visual>
@@ -40,5 +40,5 @@
         <origin xyz="0.02 -0.03 0" rpy="1.57 0 1.57" />
         <geometry>
-           <mesh filename="package://mm_description/meshes/mobile_base/asus_xtion_pro_live_camera.dae" scale="0.001 0.001 0.001"/>
+           <mesh filename="package://mm_description/meshes/sensors/asus_xtion_pro_live_camera.dae" scale="0.001 0.001 0.001"/>
         </geometry>
       </collision >

Commit message: add gazebo plugins for asus camera, but the pose of the pose of camera shot is not right.(AIMM-PC)

File: mm_description/urdf/mobile_manipulator.urdf.xacro (robot description, xacro)
@@ -4,20 +4,13 @@
   <property name="arm_prefix" value="arm_" /> <!-- I need name mobile base as base_link for navigation, so it will conflict with ur base link if prefix is not set. -->
   <!-- common stuff -->
-  <xacro:include filename="$(find mm_description)/urdf/common.gazebo" />
+  <xacro:include filename="$(find mm_description)/urdf/mobile_manipulator.gazebo.xacro" />
   <!-- ur5 -->
   <xacro:include filename="$(find mm_description)/urdf/ur5/ur5.urdf.xacro" />
   <!-- mobile base -->
   <xacro:include filename="$(find mm_description)/urdf/mobile_base/mobile_base.xacro" />
+  <!--xacro:include filename="$(find mm_description)/urdf/sensors/asus_xtion_camera.urdf.xacro" /-->
   <!-- arm -->
   <xacro:ur5_robot prefix="${arm_prefix}" joint_limited="true"/>
   <xacro:mobile_base />
-<!--
-  <link name="world" />
-  <joint name="world_2_base_link" type="fixed">
-    <parent link="world" />
-    <child link = "base_link" />
-    <origin xyz="0.0 0.0 0.0" rpy="0.0 0.0 0.0" />
-  </joint>
-  -->
   <joint name="base_link_2_${arm_prefix}base_link" type="fixed">
     <parent link="base_link" />
@@ -25,5 +18,8 @@
     <origin xyz="0.40 0 0.823" rpy="0 0 -1.5708" />
   </joint>
-  <link name="xtion_link">
+  <!--xacro:asus_xtion_camera name="xtion1" parent="${arm_prefix}base_link" tilt="0">
+    <origin xyz="-0.2841575 0.0807695 0.779517" rpy="-0.369 0.825 1.119"/>
+  </xacro:asus_xtion_camera-->
+  <link name="xtion1_frame">
       <inertial>
         <mass value="1e-5" />
@@ -44,8 +40,9 @@
       </collision >
   </link>
-  <joint name="${arm_prefix}base_link_2_xtion_link" type="fixed">
+  <joint name="${arm_prefix}base_link_2_xtion1_frame" type="fixed">
 	<parent link="${arm_prefix}base_link"/>
-	<child link="xtion_link"/>
+	<child link="xtion1_frame"/>
 	<origin xyz="-0.3541575 0.1507695 0.779517" rpy="-0.369 0.825 1.119"/>
   </joint>
+  <xacro:kinect_camera_gazebo_v0 name="xtion1" />
 </robot>

File: mm_description/urdf/sensors/asus_xtion_camera.urdf.xacro (robot description, xacro)
@@ -1,7 +1,8 @@
 <?xml version="1.0"?>
-<root xmlns:xacro="http://playerstage.sourceforge.net/gazebo/xmlschema/#interface">
+<robot xmlns:xacro="http://ros.org/wiki/xacro">
   <xacro:include filename="$(find mm_description)/urdf/sensors/asus_xtion_camera.gazebo.xacro" />
   <property name="eye_x_offset" value="0.03" />
   <property name="eye_y_offset" value="0.035" />
+  <property name="M_PI" value="3.1415926" />
   <xacro:macro name="asus_xtion_eye" params="suffix parent *origin">
 	<link name="${parent}_${suffix}_frame">
@@ -9,5 +10,5 @@
 		<mass value="0.01" />
 		<origin xyz="0 0 0" />
-		<inertia ixx="0.1" ixy="0" ixz="0" iyy="0.1" iyz="0" izz="0.1" />
+		<inertia ixx="0.0001" ixy="0" ixz="0" iyy="0.0001" iyz="0" izz="0.0001" />
 	  </inertial>
 	</link>
@@ -37,5 +38,5 @@
            <mesh filename="package://mm_description/meshes/sensors/asus_xtion_pro_live_base.dae" scale="0.0004 0.0007 0.001"/>
         </geometry>
-      </collision >
+      </collisi>
     </link>
     <joint name="${name}_foot_joint" type="fixed">
@@ -118,3 +119,3 @@
    <xacro:asus_xtion_camera_gazebo name="${name}" />
   </xacro:macro>
-</root>
+</robot>

Commit message: add some meshes

File: mm_description/urdf/mobile_manipulator.urdf.xacro (robot description, xacro)
@@ -27,6 +27,6 @@
         <inertia ixx="1e-6" ixy="0" ixz="0" iyy="1e-6" iyz="0" izz="1e-6" />
       </inertial>
-      <!--visual>
-        <origin xyz="0.02 -0.03 0" rpy="1.57 0 1.57" />
+      <visual>
+        <origin xyz="0.0 0.0 0" rpy="1.57 0 1.57" />
         <geometry>
           <mesh filename="package://mm_description/meshes/sensors/asus_xtion_pro_live_camera.dae" scale="0.001 0.001 0.001"/>
@@ -34,14 +34,14 @@
       </visual>
       <collision>
-        <origin xyz="0.02 -0.03 0" rpy="1.57 0 1.57" />
+        <origin xyz="0.0 0.0 0" rpy="1.57 0 1.57" />
         <geometry>
            <mesh filename="package://mm_description/meshes/sensors/asus_xtion_pro_live_camera.dae" scale="0.001 0.001 0.001"/>
         </geometry>
-      </collision-->
+      </collision>
   </link>
   <joint name="${arm_prefix}base_link_2_xtion1_frame" type="fixed">
 	<parent link="${arm_prefix}base_link"/>
 	<child link="xtion1_frame"/>
-	<origin xyz="-0.3541575 0.1507695 0.779517" rpy="-0.369 0.825 1.119"/>
+	<origin xyz="-0.2741575 0.0807695 0.779517" rpy="-0.369 0.825 1.119"/>
   </joint>
   <joint name="xtion1_frame_2_xtion1_optical_frame" type="fixed">

Commit message: add robotiq gripper, but there are conflicts when using position controller and velocity controller together.

File: mm_description/urdf/mobile_manipulator.urdf.xacro (robot description, xacro)
@@ -3,4 +3,5 @@
        name="mm" >
   <property name="arm_prefix" value="arm_" /> <!-- I need name mobile base as base_link for navigation, so it will conflict with ur base link if prefix is not set. -->
+  <property name="PI" value="3.1415926" />
   <!-- common stuff -->
   <xacro:include filename="$(find mm_description)/urdf/mobile_manipulator.gazebo.xacro" />
@@ -9,5 +10,6 @@
   <!-- mobile base -->
   <xacro:include filename="$(find mm_description)/urdf/mobile_base/mobile_base.xacro" />
-  <!--xacro:include filename="$(find mm_description)/urdf/sensors/asus_xtion_camera.urdf.xacro" /-->
+  <!-- gripper -->
+  <xacro:include filename="$(find robotiq_85_description)/urdf/mm_robotiq_85_gripper.urdf.xacro" />
   <!-- arm -->
   <xacro:ur5_robot prefix="${arm_prefix}" joint_limited="true"/>
@@ -18,7 +20,7 @@
     <origin xyz="0.40 0 0.823" rpy="0 0 -1.5708" />
   </joint>
-  <!--xacro:asus_xtion_camera name="xtion1" parent="${arm_prefix}base_link" tilt="0">
-    <origin xyz="-0.2841575 0.0807695 0.779517" rpy="-0.369 0.825 1.119"/>
-  </xacro:asus_xtion_camera-->
+  <xacro:robotiq_85_gripper prefix="" parent="${arm_prefix}tool0" >
+      <origin xyz="0.0 0 0.0" rpy="0 ${-PI/2} 0"/>
+  </xacro:robotiq_85_gripper>
   <link name="xtion1_frame">
       <inertial>

File: mm_description/urdf/mobile_manipulator_vel_control.urdf.xacro (robot description, xacro)
@@ -3,4 +3,5 @@
        name="mm" >
   <property name="arm_prefix" value="arm_" /> <!-- I need name mobile base as base_link for navigation, so it will conflict with ur base link if prefix is not set. -->
+  <property name="PI" value="3.1415926" />
   <!-- common stuff -->
   <xacro:include filename="$(find mm_description)/urdf/mobile_manipulator_vel_control.gazebo.xacro" />
@@ -9,8 +10,12 @@
   <!-- mobile base -->
   <xacro:include filename="$(find mm_description)/urdf/mobile_base/mobile_base_vel_control.xacro" />
-  <!--xacro:include filename="$(find mm_description)/urdf/sensors/asus_xtion_camera.urdf.xacro" /-->
+  <!-- gripper -->
+  <xacro:include filename="$(find robotiq_85_description)/urdf/mm_robotiq_85_gripper.urdf.xacro" />
   <!-- arm -->
   <xacro:ur5_robot prefix="${arm_prefix}" joint_limited="true"/>
   <xacro:mobile_base />
+  <xacro:robotiq_85_gripper prefix="" parent="${arm_prefix}tool0" >
+      <origin xyz="0.0 0 0.0" rpy="0 ${-PI/2} 0"/>
+  </xacro:robotiq_85_gripper>
   <joint name="base_link_2_${arm_prefix}base_link" type="fixed">
     <parent link="base_link" />
@@ -18,7 +23,4 @@
     <origin xyz="0.40 0 0.823" rpy="0 0 -1.5708" />
   </joint>
-  <!--xacro:asus_xtion_camera name="xtion1" parent="${arm_prefix}base_link" tilt="0">
-    <origin xyz="-0.2841575 0.0807695 0.779517" rpy="-0.369 0.825 1.119"/>
-  </xacro:asus_xtion_camera-->
   <link name="xtion1_frame">
       <inertial>

File: mm_description/urdf/ur5/ur5.urdf.xacro (robot description, xacro)
@@ -207,5 +207,5 @@
         </geometry>
       </collision>
-      <xacro:cylinder_inertial radius="0.6" length="0.12" mass="${wrist_1_mass}">
+      <xacro:cylinder_inertial radius="0.06" length="0.12" mass="${wrist_1_mass}">
         <origin xyz="0.0 0.0 0.0" rpy="0 0 0" />
       </xacro:cylinder_inertial>
@@ -238,5 +238,5 @@
         </geometry>
       </collision>
-      <xacro:cylinder_inertial radius="0.6" length="0.12" mass="${wrist_2_mass}">
+      <xacro:cylinder_inertial radius="0.06" length="0.12" mass="${wrist_2_mass}">
         <origin xyz="0.0 0.0 0.0" rpy="0 0 0" />
       </xacro:cylinder_inertial>
@@ -269,5 +269,5 @@
         </geometry>
       </collision>
-      <xacro:cylinder_inertial radius="0.6" length="0.12" mass="${wrist_3_mass}">
+      <xacro:cylinder_inertial radius="0.06" length="0.12" mass="${wrist_3_mass}">
         <origin xyz="0.0 0.0 0.0" rpy="0 0 0" />
       </xacro:cylinder_inertial>
