Commit message: re-generate mm_moveit_config package, some problem with self-collision

File: mm_description/urdf/mobile_manipulator.urdf (robot description, URDF)
Before this commit: robot mm, 17 links, 16 joints
Links:
- added link robotiq_85_base_link, mass 0.636951; collision mesh filename=package://robotiq_85_description/meshes/collision/robotiq_8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; visual mesh filename=package://robotiq_85_description/meshes/visual/robotiq_85_b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
- added link robotiq_85_left_finger_link, mass 0.027309; collision mesh filename=package://robotiq_85_description/meshes/collision/robotiq_8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; visual mesh filename=package://robotiq_85_description/meshes/visual/robotiq_85_f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
- added link robotiq_85_left_finger_tip_link, mass 0.019555; collision mesh filename=package://robotiq_85_description/meshes/collision/robotiq_8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; visual mesh filename=package://robotiq_85_description/meshes/visual/robotiq_85_f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
- added link robotiq_85_left_inner_knuckle_link, mass 0.029951; collision mesh filename=package://robotiq_85_description/meshes/collision/robotiq_8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; visual mesh filename=package://robotiq_85_description/meshes/visual/robotiq_85_i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
- added link robotiq_85_left_knuckle_link, mass 0.018491; collision mesh filename=package://robotiq_85_description/meshes/collision/robotiq_8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; visual mesh filename=package://robotiq_85_description/meshes/visual/robotiq_85_k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
- added link robotiq_85_right_finger_link, mass 0.027309; collision mesh filename=package://robotiq_85_description/meshes/collision/robotiq_8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; visual mesh filename=package://robotiq_85_description/meshes/visual/robotiq_85_f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
- added link robotiq_85_right_finger_tip_link, mass 0.019555; collision mesh filename=package://robotiq_85_description/meshes/collision/robotiq_8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; visual mesh filename=package://robotiq_85_description/meshes/visual/robotiq_85_f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
- added link robotiq_85_right_inner_knuckle_link, mass 0.029951; collision mesh filename=package://robotiq_85_description/meshes/collision/robotiq_8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; visual mesh filename=package://robotiq_85_description/meshes/visual/robotiq_85_i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
- added link robotiq_85_right_knuckle_link, mass 0.018491; collision mesh filename=package://robotiq_85_description/meshes/collision/robotiq_8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; visual mesh filename=package://robotiq_85_description/meshes/visual/robotiq_85_k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
- added link xtion1_optical_frame
- link base_link: mass 137.35 -> 1370.35
- link xtion1_frame: geometry collision mesh filename=package://mm_description/meshes/sensors/asus_xtion_pro_live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 scale=0.001 0.001 0.001; visual mesh filename=package://mm_description/meshes/sensors/asus_xtion_pro_live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 scale=0.001 0.001 0.001
Joints:
- added joint robotiq_85_base_joint: type fixed, parent arm_tool0, child robotiq_85_base_link, origin xyz=0.0 0 0.005 rpy=0 -1.5707963 0
- added joint robotiq_85_left_finger_joint: type fixed, parent robotiq_85_left_knuckle_link, child robotiq_85_left_finger_link, origin xyz=-0.00408552455 -0.03148604435 0.0 rpy=0 0 0
- added joint robotiq_85_left_finger_tip_joint: type continuous, parent robotiq_85_left_inner_knuckle_link, child robotiq_85_left_finger_tip_link, origin xyz=0.04303959807 -0.03759940821 0.0 rpy=0.0 0.0 0.0, axis 0 0 1, limit lower=-3.14 upper=3.14 effort=0.1 velocity=100.0, mimic joint=robotiq_85_left_knuckle_joint multiplier=-1
- added joint robotiq_85_left_inner_knuckle_joint: type continuous, parent robotiq_85_base_link, child robotiq_85_left_inner_knuckle_link, origin xyz=0.06142 0.0127 0 rpy=3.14159 0.0 0.0, axis 0 0 1, limit lower=-3.14 upper=3.14 effort=0.1 velocity=100.0, mimic joint=robotiq_85_left_knuckle_joint offset=0
- added joint robotiq_85_left_knuckle_joint: type revolute, parent robotiq_85_base_link, child robotiq_85_left_knuckle_link, origin xyz=0.05490451627 0.03060114443 0.0 rpy=3.14159 0.0 0.0, axis 0 0 1, limit lower=0.0 upper=0.804 effort=1000 velocity=2.0
- added joint robotiq_85_right_finger_joint: type fixed, parent robotiq_85_right_knuckle_link, child robotiq_85_right_finger_link, origin xyz=-0.00408552455 -0.03148604435 0.0 rpy=0 0 0
- added joint robotiq_85_right_finger_tip_joint: type continuous, parent robotiq_85_right_inner_knuckle_link, child robotiq_85_right_finger_tip_link, origin xyz=0.04303959807 -0.03759940821  0.0 rpy=0.0 0.0 0.0, axis 0 0 1, limit lower=-3.14 upper=3.14 effort=0.1 velocity=100.0, mimic joint=robotiq_85_left_knuckle_joint multiplier=-1
- added joint robotiq_85_right_inner_knuckle_joint: type continuous, parent robotiq_85_base_link, child robotiq_85_right_inner_knuckle_link, origin xyz=0.06142 -0.0127 0 rpy=0 0 0, axis 0 0 1, limit lower=-3.14 upper=3.14 effort=0.1 velocity=100.0, mimic joint=robotiq_85_left_knuckle_joint offset=0
- added joint robotiq_85_right_knuckle_joint: type continuous, parent robotiq_85_base_link, child robotiq_85_right_knuckle_link, origin xyz=0.05490451627 -0.03060114443 0.0 rpy=0.0 0.0 0.0, axis 0 0 1, limit lower=-3.14 upper=3.14 effort=1000 velocity=100.0, mimic joint=robotiq_85_left_knuckle_joint
- added joint xtion1_frame_2_xtion1_optical_frame: type fixed, parent xtion1_frame, child xtion1_optical_frame, origin xyz=0 0 0 rpy=-1.5707963 0 -1.5707963
- joint arm_base_link-base_fixed_joint: origin xyz=0 0 0 rpy=0 0 -3.14159265 -> xyz=0 0 0 rpy=0 0 -3.14159
- joint arm_base_link_2_xtion1_frame: origin xyz=-0.3541575 0.1507695 0.779517 rpy=-0.369 0.825 1.119 -> xyz=-0.2741575 0.0807695 0.779517 rpy=-0.369 0.825 1.119
- joint arm_ee_fixed_joint: origin xyz=0.0 0.0823 0.0 rpy=0.0 0.0 1.570796325 -> xyz=0.0 0.0823 0.0 rpy=0.0 0.0 1.570795
- joint arm_elbow_joint: limit lower=-3.14159265 upper=3.14159265 effort=150.0 velocity=3.15 -> lower=-3.14159 upper=3.14159 effort=150.0 velocity=3.15
- joint arm_shoulder_lift_joint: limit lower=-3.14159265 upper=3.14159265 effort=150.0 velocity=3.15 -> lower=-3.14159 upper=3.14159 effort=150.0 velocity=3.15; origin xyz=0.0 0.13585 0.0 rpy=0.0 1.570796325 0.0 -> xyz=0.0 0.13585 0.0 rpy=0.0 1.570795 0.0
- joint arm_shoulder_pan_joint: limit lower=-3.14159265 upper=3.14159265 effort=150.0 velocity=3.15 -> lower=-3.14159 upper=3.14159 effort=150.0 velocity=3.15
- joint arm_wrist_1_joint: limit lower=-3.14159265 upper=3.14159265 effort=28.0 velocity=3.2 -> lower=-3.14159 upper=3.14159 effort=28.0 velocity=3.2; origin xyz=0.0 0.0 0.39225 rpy=0.0 1.570796325 0.0 -> xyz=0.0 0.0 0.39225 rpy=0.0 1.570795 0.0
- joint arm_wrist_2_joint: limit lower=-3.14159265 upper=3.14159265 effort=28.0 velocity=3.2 -> lower=-3.14159 upper=3.14159 effort=28.0 velocity=3.2
- joint arm_wrist_3_joint: limit lower=-3.14159265 upper=3.14159265 effort=28.0 velocity=3.2 -> lower=-3.14159 upper=3.14159 effort=28.0 velocity=3.2
- joint arm_wrist_3_link-tool0_fixed_joint: origin xyz=0 0.0823 0 rpy=-1.570796325 0 0 -> xyz=0 0.0823 0 rpy=-1.570795 0 0

File: mm_description/urdf/mobile_manipulator.urdf.xacro (robot description, xacro)
@@ -21,5 +21,5 @@
   </joint>
   <xacro:robotiq_85_gripper prefix="" parent="${arm_prefix}tool0" >
-      <origin xyz="0.0 0 0.0" rpy="0 ${-PI/2} 0"/>
+      <origin xyz="0.0 0 0.005" rpy="0 ${-PI/2} 0"/>
   </xacro:robotiq_85_gripper>
   <link name="xtion1_frame">
