Commit message: add package mm_ar_track, which is used to track ar code.(AIMM-PC)

File: mm_gazebo/urdf/room100.urdf.xacro (robot description, xacro)
@@ -2,4 +2,5 @@
 <robot xmlns:xacro="http://www.ros.org/wiki/xacro"
        name="room100" >
+    <property name="M_PI" value="3.1415926" />
     <link name="wall">
         <inertial>
@@ -24,5 +25,5 @@
         <parent link="wall" />
         <child link="qr_board1" />
-        <origin xyz="13 1.24 1" rpy="0 0 0" />
+        <origin xyz="13 1.54 1" rpy="0 0 0" />
     </joint>
     <link name="qr_board1">
@@ -48,5 +49,5 @@
         <parent link="wall" />
         <child link="qr_board2" />
-        <origin xyz="14.135 11.265 1" rpy="0 0 0" />
+        <origin xyz="14.135 11.265 1" rpy="0 0 ${M_PI/2}" />
     </joint>
     <link name="qr_board2">

Commit message: add two air-conditions

File: mm_gazebo/urdf/room100.urdf.xacro (robot description, xacro)
@@ -3,4 +3,5 @@
        name="room100" >
     <property name="M_PI" value="3.1415926" />
+    <!-- wall of room 100 -->
     <link name="wall">
         <inertial>
@@ -22,4 +23,104 @@
         </collision>
     </link>
+    <joint name="wall_2_long_desk1" type="fixed">
+        <parent link="wall" />
+        <child link="long_desk1" />
+        <origin xyz="4 3 0" rpy="0 0 0" />
+    </joint>
+    <!-- long desk 1 -->
+    <link name="long_desk1">
+        <inertial>
+          <origin xyz="0 0 0" />
+          <mass value="10000000.0" />
+          <inertia  ixx="1000000.0" ixy="0.0"  ixz="0.0"  iyy="1000000.0"  iyz="0.0"  izz="1000000.0" />
+        </inertial>
+        <visual>
+          <origin xyz="0 0 0"/>
+          <geometry>
+            <mesh filename="package://mm_gazebo/meshes/longdesk.dae" />
+          </geometry>
+        </visual>
+        <collision>
+          <origin xyz="0 0 0"/>
+          <geometry>
+            <mesh filename="package://mm_gazebo/meshes/longdesk.dae" />
+          </geometry>
+        </collision>
+    </link>
+    <joint name="wall_2_long_desk2" type="fixed">
+        <parent link="wall" />
+        <child link="long_desk2" />
+        <origin xyz="4 3.58 0" rpy="0 0 0" />
+    </joint>
+    <!-- long desk 2 -->
+    <link name="long_desk2">
+        <inertial>
+          <origin xyz="0 0 0" />
+          <mass value="10000000.0" />
+          <inertia  ixx="1000000.0" ixy="0.0"  ixz="0.0"  iyy="1000000.0"  iyz="0.0"  izz="1000000.0" />
+        </inertial>
+        <visual>
+          <origin xyz="0 0 0"/>
+          <geometry>
+            <mesh filename="package://mm_gazebo/meshes/longdesk.dae" />
+          </geometry>
+        </visual>
+        <collision>
+          <origin xyz="0 0 0"/>
+          <geometry>
+            <mesh filename="package://mm_gazebo/meshes/longdesk.dae" />
+          </geometry>
+        </collision>
+    </link>
+    <joint name="wall_2_aircon1" type="fixed">
+        <parent link="wall" />
+        <child link="aircon1" />
+        <origin xyz="0.4 0.4 0" rpy="${M_PI/2} 0 ${-M_PI/4}" />
+    </joint>
+    <!-- air condition 1 -->
+    <link name="aircon1">
+        <inertial>
+          <origin xyz="0 0 0" />
+          <mass value="10000000.0" />
+          <inertia  ixx="1000000.0" ixy="0.0"  ixz="0.0"  iyy="1000000.0"  iyz="0.0"  izz="1000000.0" />
+        </inertial>
+        <visual>
+          <origin xyz="0 0 0"/>
+          <geometry>
+            <mesh filename="package://mm_gazebo/meshes/aircon.dae" />
+          </geometry>
+        </visual>
+        <collision>
+          <origin xyz="0 0 0"/>
+          <geometry>
+            <mesh filename="package://mm_gazebo/meshes/aircon.dae" />
+          </geometry>
+        </collision>
+    </link>
+    <joint name="wall_2_aircon2" type="fixed">
+        <parent link="wall" />
+        <child link="aircon2" />
+        <origin xyz="0.4 11.7 0" rpy="${M_PI/2} 0 ${-3*M_PI/4}" />
+    </joint>
+    <!-- air condition 1 -->
+    <link name="aircon2">
+        <inertial>
+          <origin xyz="0 0 0" />
+          <mass value="10000000.0" />
+          <inertia  ixx="1000000.0" ixy="0.0"  ixz="0.0"  iyy="1000000.0"  iyz="0.0"  izz="1000000.0" />
+        </inertial>
+        <visual>
+          <origin xyz="0 0 0"/>
+          <geometry>
+            <mesh filename="package://mm_gazebo/meshes/aircon.dae" />
+          </geometry>
+        </visual>
+        <collision>
+          <origin xyz="0 0 0"/>
+          <geometry>
+            <mesh filename="package://mm_gazebo/meshes/aircon.dae" />
+          </geometry>
+        </collision>
+    </link>
     <joint name="wall_2_qr_board1" type="fixed">
         <parent link="wall" />
@@ -27,4 +128,5 @@
         <origin xyz="13 1.54 1" rpy="0 0 0" />
     </joint>
+    <!-- qr board on desk 1 -->
     <link name="qr_board1">
         <inertial>
@@ -51,4 +153,5 @@
         <origin xyz="14.135 11.265 1" rpy="0 0 ${M_PI/2}" />
     </joint>
+    <!-- qr board on desk 2 -->
     <link name="qr_board2">
         <inertial>

Commit message: add a lot of things in room 100

File: mm_gazebo/urdf/room100.urdf.xacro (robot description, xacro)
@@ -3,4 +3,7 @@
        name="room100" >
     <property name="M_PI" value="3.1415926" />
+    <xacro:include filename="$(find mm_gazebo)/urdf/materials.xacro" />
+    <xacro:include filename="$(find mm_gazebo)/urdf/room100.gazebo.xacro" />
+    <xacro:room100_gazebo />
     <!-- wall of room 100 -->
     <link name="wall">
@@ -123,4 +126,180 @@
         </collision>
     </link>
+    <joint name="wall_2_workdesk1" type="fixed">
+        <parent link="wall" />
+        <child link="workdesk1" />
+        <origin xyz="2.4 11.6 0" rpy="${M_PI/2} 0 ${M_PI}" />
+    </joint>
+    <!-- work desk 1 -->
+    <link name="workdesk1">
+        <inertial>
+          <origin xyz="0 0 0" />
+          <mass value="10000000.0" />
+          <inertia  ixx="1000000.0" ixy="0.0"  ixz="0.0"  iyy="1000000.0"  iyz="0.0"  izz="1000000.0" />
+        </inertial>
+        <visual>
+          <origin xyz="0 0 0"/>
+          <geometry>
+            <mesh filename="package://mm_gazebo/meshes/workdesk.dae" />
+          </geometry>
+        </visual>
+        <collision>
+          <origin xyz="0 0 0"/>
+          <geometry>
+            <mesh filename="package://mm_gazebo/meshes/workdesk.dae" />
+          </geometry>
+        </collision>
+    </link>
+    <joint name="wall_2_workdesk2" type="fixed">
+        <parent link="wall" />
+        <child link="workdesk2" />
+        <origin xyz="4.4 11.6 0" rpy="${M_PI/2} 0 ${M_PI}" />
+    </joint>
+    <!-- work desk 2 -->
+    <link name="workdesk2">
+        <inertial>
+          <origin xyz="0 0 0" />
+          <mass value="10000000.0" />
+          <inertia  ixx="1000000.0" ixy="0.0"  ixz="0.0"  iyy="1000000.0"  iyz="0.0"  izz="1000000.0" />
+        </inertial>
+        <visual>
+          <origin xyz="0 0 0"/>
+          <geometry>
+            <mesh filename="package://mm_gazebo/meshes/workdesk.dae" />
+          </geometry>
+        </visual>
+        <collision>
+          <origin xyz="0 0 0"/>
+          <geometry>
+            <mesh filename="package://mm_gazebo/meshes/workdesk.dae" />
+          </geometry>
+        </collision>
+    </link>
+    <joint name="wall_2_workdesk3" type="fixed">
+        <parent link="wall" />
+        <child link="workdesk3" />
+        <origin xyz="0.4 8.6 0" rpy="${M_PI/2} 0 ${-M_PI/2}" />
+    </joint>
+    <!-- work desk 3 -->
+    <link name="workdesk3">
+        <inertial>
+          <origin xyz="0 0 0" />
+          <mass value="10000000.0" />
+          <inertia  ixx="1000000.0" ixy="0.0"  ixz="0.0"  iyy="1000000.0"  iyz="0.0"  izz="1000000.0" />
+        </inertial>
+        <visual>
+          <origin xyz="0 0 0"/>
+          <geometry>
+            <mesh filename="package://mm_gazebo/meshes/workdesk.dae" />
+          </geometry>
+        </visual>
+        <collision>
+          <origin xyz="0 0 0"/>
+          <geometry>
+            <mesh filename="package://mm_gazebo/meshes/workdesk.dae" />
+          </geometry>
+        </collision>
+    </link>
+    <joint name="wall_2_storage" type="fixed">
+        <parent link="wall" />
+        <child link="storage" />
+        <origin xyz="6 3.3 0.75" rpy="0 0 ${-M_PI/2}" />
+    </joint>
+    <!-- storage -->
+    <link name="storage">
+        <inertial>
+          <origin xyz="0 0 0" />
+          <mass value="10000000.0" />
+          <inertia  ixx="1000000.0" ixy="0.0"  ixz="0.0"  iyy="1000000.0"  iyz="0.0"  izz="1000000.0" />
+        </inertial>
+        <visual>
+          <origin xyz="0 0 0"/>
+          <geometry>
+            <mesh filename="package://mm_gazebo/meshes/storage.dae" />
+          </geometry>
+        </visual>
+        <collision>
+          <origin xyz="0 0 0"/>
+          <geometry>
+            <mesh filename="package://mm_gazebo/meshes/storage.dae" />
+          </geometry>
+        </collision>
+    </link>
+    <joint name="wall_2_elevbox" type="fixed">
+        <parent link="wall" />
+        <child link="elevbox" />
+        <origin xyz="7.5 11.7 0" rpy="0 0 0" />
+    </joint>
+    <!-- elevator box 1 -->
+    <link name="elevbox">
+        <inertial>
+          <origin xyz="0 0 0" />
+          <mass value="10000000.0" />
+          <inertia  ixx="1000000.0" ixy="0.0"  ixz="0.0"  iyy="1000000.0"  iyz="0.0"  izz="1000000.0" />
+        </inertial>
+        <visual>
+          <origin xyz="0 0 0"/>
+          <geometry>
+            <mesh filename="package://mm_gazebo/meshes/elevator_box.dae" scale="0.4 0.4 0.4"/>
+          </geometry>
+        </visual>
+        <collision>
+          <origin xyz="0 0 0"/>
+          <geometry>
+            <mesh filename="package://mm_gazebo/meshes/elevator_box.dae" scale="0.4 0.4 0.4"/>
+          </geometry>
+        </collision>
+    </link>
+    <joint name="wall_2_desk" type="fixed">
+        <parent link="wall" />
+        <child link="desk" />
+        <origin xyz="9 11 0" rpy="0 0 ${M_PI}" />
+    </joint>
+    <!-- elevator box 1 -->
+    <link name="desk">
+        <inertial>
+          <origin xyz="0 0 0" />
+          <mass value="10000000.0" />
+          <inertia  ixx="1000000.0" ixy="0.0"  ixz="0.0"  iyy="1000000.0"  iyz="0.0"  izz="1000000.0" />
+        </inertial>
+        <visual>
+          <origin xyz="0 0 0"/>
+          <geometry>
+            <mesh filename="package://mm_gazebo/meshes/desk.stl"/>
+          </geometry>
+        </visual>
+        <collision>
+          <origin xyz="0 0 0"/>
+          <geometry>
+            <mesh filename="package://mm_gazebo/meshes/desk.stl"/>
+          </geometry>
+        </collision>
+    </link>
+    <joint name="wall_2_line" type="fixed">
+        <parent link="wall" />
+        <child link="line" />
+        <origin xyz="10 3.6 0" rpy="0 0 ${M_PI/2}" />
+    </joint>
+    <!-- line -->
+    <link name="line">
+        <inertial>
+          <origin xyz="0 0 0" />
+          <mass value="10000000.0" />
+          <inertia  ixx="1000000.0" ixy="0.0"  ixz="0.0"  iyy="1000000.0"  iyz="0.0"  izz="1000000.0" />
+        </inertial>
+        <visual>
+          <origin xyz="0 0 0"/>
+          <geometry>
+            <mesh filename="package://mm_gazebo/meshes/line.dae" />
+          </geometry>
+        </visual>
+        <collision>
+          <origin xyz="0 0 0"/>
+          <geometry>
+            <mesh filename="package://mm_gazebo/meshes/line.dae" />
+          </geometry>
+        </collision>
+    </link>
+    <!-- ############ qr boards ############### -->
     <joint name="wall_2_qr_board1" type="fixed">
         <parent link="wall" />
@@ -173,3 +352,124 @@
         </collision>
     </link>
+    <!-- ############ boxes ############### -->
+    <joint name="wall_2_box1" type="fixed">
+        <parent link="wall" />
+        <child link="box1" />
+        <origin xyz="12.4 1 0.25" rpy="0 0 0" />
+    </joint>
+    <link name="box1">
+        <inertial>
+          <origin xyz="0 0 0" />
+          <mass value="100" />
+          <inertia  ixx="1" ixy="0.0"  ixz="0.0"  iyy="1"  iyz="0.0"  izz="1" />
+        </inertial>
+        <visual>
+          <origin xyz="0 0 0"/>
+          <geometry>
+            <box size="1 1.2 0.5" />
+          </geometry>
+        </visual>
+        <collision>
+          <origin xyz="0 0 0"/>
+          <geometry>
+            <box size="1 1.5 0.5"  />
+          </geometry>
+        </collision>
+    </link>
+    <joint name="wall_2_box2" type="fixed">
+        <parent link="wall" />
+        <child link="box2" />
+        <origin xyz="10 5 0.25" rpy="0 0 0" />
+    </joint>
+    <link name="box2">
+        <inertial>
+          <origin xyz="0 0 0" />
+          <mass value="100" />
+          <inertia  ixx="1" ixy="0.0"  ixz="0.0"  iyy="1"  iyz="0.0"  izz="1" />
+        </inertial>
+        <visual>
+          <origin xyz="0 0 0"/>
+          <geometry>
+            <box size="0.5 1.2 0.5" />
+          </geometry>
+        </visual>
+        <collision>
+          <origin xyz="0 0 0"/>
+          <geometry>
+            <box size="0.5 1.5 0.5"  />
+          </geometry>
+        </collision>
+    </link>
+    <joint name="wall_2_box3" type="fixed">
+        <parent link="wall" />
+        <child link="box3" />
+        <origin xyz="9.8 6.5 0.25" rpy="0 0 0" />
+    </joint>
+    <link name="box3">
+        <inertial>
+          <origin xyz="0 0 0" />
+          <mass value="100" />
+          <inertia  ixx="1" ixy="0.0"  ixz="0.0"  iyy="1"  iyz="0.0"  izz="1" />
+        </inertial>
+        <visual>
+          <origin xyz="0 0 0"/>
+          <geometry>
+            <box size="0.5 1.5 0.5" />
+          </geometry>
+        </visual>
+        <collision>
+          <origin xyz="0 0 0"/>
+          <geometry>
+            <box size="0.5 1.5 0.5"  />
+          </geometry>
+        </collision>
+    </link>
+    <joint name="wall_2_box4" type="fixed">
+        <parent link="wall" />
+        <child link="box4" />
+        <origin xyz="5.5 3.2 0.25" rpy="0 0 0" />
+    </joint>
+    <link name="box4">
+        <inertial>
+          <origin xyz="0 0 0" />
+          <mass value="100" />
+          <inertia  ixx="1" ixy="0.0"  ixz="0.0"  iyy="1"  iyz="0.0"  izz="1" />
+        </inertial>
+        <visual>
+          <origin xyz="0 0 0"/>
+          <geometry>
+            <box size="1 0.8 0.5" />
+          </geometry>
+        </visual>
+        <collision>
+          <origin xyz="0 0 0"/>
+          <geometry>
+            <box size="1 0.8 0.5"  />
+          </geometry>
+        </collision>
+    </link>
+    <joint name="wall_2_box5" type="fixed">
+        <parent link="wall" />
+        <child link="box5" />
+        <origin xyz="4 3 0.25" rpy="0 0 0" />
+    </joint>
+    <link name="box5">
+        <inertial>
+          <origin xyz="0 0 0" />
+          <mass value="100" />
+          <inertia  ixx="1" ixy="0.0"  ixz="0.0"  iyy="1"  iyz="0.0"  izz="1" />
+        </inertial>
+        <visual>
+          <origin xyz="0 0 0"/>
+          <geometry>
+            <box size="1.5 0.6 0.5" />
+          </geometry>
+        </visual>
+        <collision>
+          <origin xyz="0 0 0"/>
+          <geometry>
+            <box size="1.5 0.6 0.5"  />
+          </geometry>
+        </collision>
+    </link>
 </robot>

Commit message: add mm_navigation and the map of room 100

File: mm_gazebo/urdf/room100.urdf.xacro (robot description, xacro)
@@ -301,4 +301,29 @@
         </collision>
     </link>
+    <joint name="wall_2_shelf" type="fixed">
+        <parent link="wall" />
+        <child link="shelf" />
+        <origin xyz="0.2 1.6 0" rpy="${M_PI/2} 0 ${M_PI/2}" />
+    </joint>
+    <!-- line -->
+    <link name="shelf">
+        <inertial>
+          <origin xyz="0 0 0" />
+          <mass value="10000000.0" />
+          <inertia  ixx="1000000.0" ixy="0.0"  ixz="0.0"  iyy="1000000.0"  iyz="0.0"  izz="1000000.0" />
+        </inertial>
+        <visual>
+          <origin xyz="0 0 0"/>
+          <geometry>
+            <mesh filename="package://mm_gazebo/meshes/shelf.dae" />
+          </geometry>
+        </visual>
+        <collision>
+          <origin xyz="0 0 0"/>
+          <geometry>
+            <mesh filename="package://mm_gazebo/meshes/shelf.dae" />
+          </geometry>
+        </collision>
+    </link>
     <!-- ############ qr boards ############### -->
     <joint name="wall_2_qr_board1" type="fixed">
@@ -352,4 +377,29 @@
         </collision>
     </link>
+    <joint name="wall_2_qr_board3" type="fixed">
+        <parent link="wall" />
+        <child link="qr_board3" />
+        <origin xyz="9.3 10.8 0.7" rpy="0 0 ${M_PI}" />
+    </joint>
+    <!-- qr board on desk 3 -->
+    <link name="qr_board3">
+        <inertial>
+          <origin xyz="0 0 0" />
+          <mass value="0.01" />
+          <inertia  ixx="0.00001" ixy="0.0"  ixz="0.0"  iyy="0.00001"  iyz="0.0"  izz="0.00001" />
+        </inertial>
+        <visual>
+          <origin xyz="0 0 0"/>
+          <geometry>
+            <mesh filename="package://mm_gazebo/meshes/qr_board.dae" />
+          </geometry>
+        </visual>
+        <collision>
+          <origin xyz="0 0 0"/>
+          <geometry>
+            <mesh filename="package://mm_gazebo/meshes/qr_board.dae" />
+          </geometry>
+        </collision>
+    </link>
     <!-- ############ boxes ############### -->
     <joint name="wall_2_box1" type="fixed">
