Commit message: modify the mm_robotiq_85_gripper.urdf.xacro, and set all the joint to fix

File: robotiq_85_gripper/robotiq_85_description/urdf/mm_robotiq_85_gripper.urdf.xacro (robot description, xacro)
@@ -1,5 +1,5 @@
 <?xml version="1.0"?>
 <robot name="robotiq_85_gripper" xmlns:xacro="http://ros.org/wiki/xacro">
-    <xacro:include filename="$(find robotiq_85_description)/urdf/mm_robotiq_85_gripper.transmission.xacro" />
+    <!--xacro:include filename="$(find robotiq_85_description)/urdf/mm_robotiq_85_gripper.transmission.xacro" /-->
     <property name="pi" value="3.14159"/>
     <xacro:macro name="robotiq_85_gripper" params="prefix parent *origin">
@@ -28,5 +28,5 @@
             </inertial>
         </link>
-        <joint name="${prefix}robotiq_85_left_knuckle_joint" type="revolute">
+        <joint name="${prefix}robotiq_85_left_knuckle_joint" type="fixed"> <!-- revolute -->
             <parent link="${prefix}robotiq_85_base_link"/>
             <child link="${prefix}robotiq_85_left_knuckle_link"/>
@@ -35,5 +35,5 @@
             <limit lower="0.0" upper="0.804" velocity="2.0" effort="1000"/>
         </joint>
-        <joint name="${prefix}robotiq_85_right_knuckle_joint" type="continuous">
+        <joint name="${prefix}robotiq_85_right_knuckle_joint" type="fixed"> <!--continuous-->
             <parent link="${prefix}robotiq_85_base_link"/>
             <child link="${prefix}robotiq_85_right_knuckle_link"/>
@@ -129,5 +129,5 @@
             </inertial>
         </link>
-        <joint name="${prefix}robotiq_85_left_inner_knuckle_joint" type="continuous">
+        <joint name="${prefix}robotiq_85_left_inner_knuckle_joint" type="fixed"> <!--continuous-->
             <parent link="${prefix}robotiq_85_base_link"/>
             <child link="${prefix}robotiq_85_left_inner_knuckle_link"/>
@@ -137,5 +137,5 @@
             <mimic joint="${prefix}robotiq_85_left_knuckle_joint" offset="0"/>
         </joint>
-        <joint name="${prefix}robotiq_85_right_inner_knuckle_joint" type="continuous">
+        <joint name="${prefix}robotiq_85_right_inner_knuckle_joint" type="fixed"> <!--continuous-->
             <parent link="${prefix}robotiq_85_base_link"/>
             <child link="${prefix}robotiq_85_right_inner_knuckle_link"/>
@@ -183,5 +183,5 @@
             </inertial>
         </link>
-        <joint name="${prefix}robotiq_85_left_finger_tip_joint" type="continuous">
+        <joint name="${prefix}robotiq_85_left_finger_tip_joint" type="fixed"> <!--continuous-->
             <parent link="${prefix}robotiq_85_left_inner_knuckle_link"/>
             <child link="${prefix}robotiq_85_left_finger_tip_link"/>
@@ -191,5 +191,5 @@
             <mimic joint="${prefix}robotiq_85_left_knuckle_joint" multiplier="-1"/>
         </joint>
-        <joint name="${prefix}robotiq_85_right_finger_tip_joint" type="continuous">
+        <joint name="${prefix}robotiq_85_right_finger_tip_joint" type="fixed"> <!--continuous-->
             <parent link="${prefix}robotiq_85_right_inner_knuckle_link"/>
             <child link="${prefix}robotiq_85_right_finger_tip_link"/>
